File: StarJar.kicad_pcb (KiCad board)
At the start: 2 copper layers, 127 x 50.8 mm, 35 parts, among them J1 USB_A, J2 GM_Tube, J3 Screw_Terminal_1x02, Q1 JN3303, Q2 2N3904, Q3 DMN1019USN-13, Q4 2N3904, U1 LM555N

Commit message: Add files via upload
v1.1 routing done and ready to order
Parts:
- removed the G*** at (178.1, 66.0)
- removed the REF*** at (116.6, 44.7)
- added G***: LOGO, KNEK-TEK_logo:KNEK-TEK_logo_11mm, F.Cu at (175.3, 63.8)
- added REF**: MountingHole_3.2mm_M3, Mounting_Holes:MountingHole_3.2mm_M3, F.Cu at (184.7, 59.7)
- added REF***: OSHW-Logo_7.5x8mm_SilkScreen, Symbols:OSHW-Logo_7.5x8mm_SilkScreen, F.Cu at (183.4, 92.5)
- added RV3: 10Ω POT, Potentiometers:Potentiometer_Trimmer_Suntan_TSR-3386P_Horizontal, F.Cu at (166.9, 95.0)
- added U2: LMV321, TO_SOT_Packages_SMD:SOT-23-5_HandSoldering, F.Cu at (164.6, 83.6)
- Q3: value DMN1019USN-13 -> 2N3904; footprint TO_SOT_Packages_SMD:SC-59_Handsoldering -> TO_SOT_Packages_THT:TO-92_Inline_Wide
- moved R2 23.6 mm to (176.0, 99.1), turned to 90 degrees
- moved C5 16.4 mm to (183.4, 70.4), turned to 90 degrees
- moved Q3 8.52 mm to (172.5, 83.6), turned to 90 degrees
- moved C4 8.18 mm to (158.8, 97.5)
- moved REF** 0.80 mm to (184.7, 100.6)
Connections:
- C5 pad 1: Net-(C5-Pad1) -> +5V
- J3 pad 2: Net-(C5-Pad1) -> +5V
- Q3 pad 1: /PulseOutput -> Net-(Q3-Pad1)
- Q3 pad 2: GND -> Net-(Q3-Pad2)
- R2 pad 1: +5V -> Net-(R2-Pad1)
- R2 pad 2: Net-(C5-Pad1) -> Net-(Q3-Pad1)
Routing:
- net +5V: track 134.4 -> 163.1 mm
- net Net-(Q3-Pad1): track 0.00 -> 19.1 mm
- net Net-(C5-Pad1): track 15.6 -> 0.00 mm
- net Net-(R2-Pad1): track 0.00 -> 10.8 mm
- net Net-(Q3-Pad2): track 0.00 -> 10.5 mm
- net GND: track 9.72 -> 17.3 mm
- net /PulseOutput: track 28.9 -> 27.9 mm
- net Net-(J3-Pad1): track 12.2 -> 13.0 mm
Other:
- net class Narrow added: clearance 0.254, trace_width 0.254, via_dia 0.6, via_drill 0.4
- board text added: "1.1"
- board text added: "LED Current Limiting"
- board text removed: "K'NEK-TEK Star Jar v1.0 Sept 2017"
- board text removed: "R2 is brightness control (5V - Vdrop) = 2.6V 2.6V / R2 = I_limit"
