File: StarJar.sch (KiCad schematic (older format))
At the start: 32 parts, among them J1 USB_A, J2 GM_Tube, J3 Screw_Terminal_1x02, Q1 JN3303, Q2 2N3904, Q3 2N3904, Q4 2N3904, U1 LM555N, U2 LMV321

Commit message: Add files via upload
v1.1 routing done and ready to order
Parts:
- U2: footprint TO_SOT_Packages_SMD:SOT-23-5 -> TO_SOT_Packages_SMD:SOT-23-5_HandSoldering
Changed lines of the file:
@@
 Geiger tube inputs
 $Comp
-L +5V #PWR1
+L +5V #PWR01
 U 1 1 59AEE24D
 P 1350 950
-F 0 "#PWR1" H 1350 800 50  0001 C CNN
+F 0 "#PWR01" H 1350 800 50  0001 C CNN
 F 1 "+5V" H 1350 1090 50  0000 C CNN
 F 2 "" H 1350 950 50  0001 C CNN
@@
 $EndComp
 $Comp
-L +5V #PWR3
+L +5V #PWR02
 U 1 1 59AEE26B
 P 2150 2950
-F 0 "#PWR3" H 2150 2800 50  0001 C CNN
+F 0 "#PWR02" H 2150 2800 50  0001 C CNN
 F 1 "+5V" H 2150 3090 50  0000 C CNN
 F 2 "" H 2150 2950 50  0001 C CNN
@@
 $EndComp
 $Comp
-L GND #PWR6
+L GND #PWR03
 U 1 1 59AEE280
 P 2150 5100
-F 0 "#PWR6" H 2150 4850 50  0001 C CNN
+F 0 "#PWR03" H 2150 4850 50  0001 C CNN
 F 1 "GND" H 2150 4950 50  0000 C CNN
 F 2 "" H 2150 5100 50  0001 C CNN
@@
 $EndComp
 $Comp
-L GND #PWR2
+L GND #PWR04
 U 1 1 59AEE29E
 P 850 1800
-F 0 "#PWR2" H 850 1550 50  0001 C CNN
+F 0 "#PWR04" H 850 1550 50  0001 C CNN
 F 1 "GND" H 850 1650 50  0000 C CNN
 F 2 "" H 850 1800 50  0001 C CNN
@@
 $EndComp
 $Comp
-L GND #PWR10
+L GND #PWR05
 U 1 1 59AF059B
 P 4200 5500
-F 0 "#PWR10" H 4200 5250 50  0001 C CNN
+F 0 "#PWR05" H 4200 5250 50  0001 C CNN
 F 1 "GND" H 4200 5350 50  0000 C CNN
 F 2 "" H 4200 5500 50  0001 C CNN
@@
 Connection ~ 6600 3500
 $Comp
-L GND #PWR7
+L GND #PWR06
 U 1 1 59AF52EC
 P 7600 5450
-F 0 "#PWR7" H 7600 5200 50  0001 C CNN
+F 0 "#PWR06" H 7600 5200 50  0001 C CNN
 F 1 "GND" H 7600 5300 50  0000 C CNN
 F 2 "" H 7600 5450 50  0001 C CNN
@@
 $EndComp
 $Comp
-L GND #PWR9
+L GND #PWR07
 U 1 1 59B08F92
 P 9850 5450
-F 0 "#PWR9" H 9850 5200 50  0001 C CNN
+F 0 "#PWR07" H 9850 5200 50  0001 C CNN
 F 1 "GND" H 9850 5300 50  0000 C CNN
 F 2 "" H 9850 5450 50  0001 C CNN
@@
 	6600 5400 8050 5400
 $Comp
-L +5V #PWR4
+L +5V #PWR08
 U 1 1 59B99BA7
 P 7600 3200
-F 0 "#PWR4" H 7600 3050 50  0001 C CNN
+F 0 "#PWR08" H 7600 3050 50  0001 C CNN
 F 1 "+5V" H 7600 3340 50  0000 C CNN
 F 2 "" H 7600 3200 50  0001 C CNN
@@
 $EndComp
 $Comp
-L GND #PWR5
+L GND #PWR09
 U 1 1 59C16D42
 P 9450 3750
-F 0 "#PWR5" H 9450 3500 50  0001 C CNN
+F 0 "#PWR09" H 9450 3500 50  0001 C CNN
 F 1 "GND" H 9450 3600 50  0000 C CNN
 F 2 "" H 9450 3750 50  0001 C CNN
@@
 Connection ~ 9450 3200
 $Comp
-L GND #PWR12
+L GND #PWR010
 U 1 1 59C172D0
 P 1350 6250
-F 0 "#PWR12" H 1350 6000 50  0001 C CNN
+F 0 "#PWR010" H 1350 6000 50  0001 C CNN
 F 1 "GND" H 1350 6100 50  0000 C CNN
 F 2 "" H 1350 6250 50  0001 C CNN
@@
 $EndComp
 $Comp
-L +5V #PWR11
+L +5V #PWR011
 U 1 1 59C17371
 P 1350 5650
-F 0 "#PWR11" H 1350 5500 50  0001 C CNN
+F 0 "#PWR011" H 1350 5500 50  0001 C CNN
 F 1 "+5V" H 1350 5790 50  0000 C CNN
 F 2 "" H 1350 5650 50  0001 C CNN
@@
 F 0 "U2" H 8850 4500 50  0000 L CNN
 F 1 "LMV321" H 8850 4100 50  0000 L CNN
-F 2 "TO_SOT_Packages_SMD:SOT-23-5" H 8850 4425 50  0001 L CNN
+F 2 "TO_SOT_Packages_SMD:SOT-23-5_HandSoldering" H 8850 4425 50  0001 L CNN
 F 3 "" H 8850 4300 50  0001 C CNN
 	1    8850 4300
@@
 	8350 4200 8350 4800
 $Comp
-L GND #PWR8
+L GND #PWR012
 U 1 1 59E556E2
 P 8750 5450
-F 0 "#PWR8" H 8750 5200 50  0001 C CNN
+F 0 "#PWR012" H 8750 5200 50  0001 C CNN
 F 1 "GND" H 8750 5300 50  0000 C CNN
 F 2 "" H 8750 5450 50  0001 C CNN

Commit message: Add files via upload
v1.2 board layout finished, ready to order. Changes: zip tie mounts for GM tube, USB micro-B rather than USB-A, added new components to fix pulse size issue.
Parts:
- removed FuseHolder1, FuseHolder2: FuseHolder, Resistors_THT:R_Axial_DIN0309_L9.0mm_D3.2mm_P15.24mm_Horizontal, symbol CONN_01X01_FEMALE
- removed J1: USB_A, Connectors:USB_A, symbol USB_A
- added J1: USB_OTG, CustomFootprints:USB_Micro-B_big_holes_for_OSHpark, symbol USB_OTG
- added Q2: 2N3906, TO_SOT_Packages_THT:TO-92_Inline_Wide, symbol Q_PNP_EBC
- added R3: 1k, Resistors_THT:R_Axial_DIN0411_L9.9mm_D3.6mm_P5.08mm_Vertical, symbol R
- added R7: 100, Resistors_THT:R_Axial_DIN0411_L9.9mm_D3.6mm_P5.08mm_Vertical, symbol R
- C1: renamed from C5; value 20uF -> 4.7uF
- C5: renamed from C4; value 20uF -> 1uF
- R6: value 22k -> 100
- RV1: value >100k POT -> 500k POT
- renumbered C1 to C2, C2 to C3, C3 to C4, J3 to J2, J2 to J3, Q2 to Q5, R8 to R10, R2 to R11, R3 to R2, R9 to R8, R7 to R9
Connections:
- net +5V: now also J1.1 (VBUS), Q2.1 (E), R3.2; no longer Q4.3 (C)
- net GND: now also Q4.1 (E), J1.5 (GND), J1.6 (Shield)
- net PulseOutput: now also R7.2; no longer Q4.1 (E)
- net at C4.1, J3.2: now also Q4.2 (B), R8.2; no longer R6.2
- new net: Q4.3 (C), R3.1, R6.1
- new net: Q2.2 (B), R6.2
- new net: Q2.3 (C), R7.1
- no-connect marks 8 -> 7
Other:
- note added: "1.2"
- note added: "StarJar Radiation Controlled Christmas Lights"
- note removed: "1.1"
- note removed: "Each fuse holder uses a 15mm spacing \nresistor footprint for mounting holes"
- note removed: "StarJar Radiation Detector"
- note removed: "Works well without R7"
- moved on the sheet: C1, C5, J2, Q3, R11, RV1, RV3, U2
